File: Hardware/Smartwatch-Jank.kicad_sch (KiCad schematic)
At the start: 10 parts, among them U1 ARDUINO_PRO_MINI

Commit message: Add new schematic with battery powering most sensors without voltage regulator
Parts:
- added 3.7_Vias1: Conn_01x02, Connector_PinHeader_2.54mm:PinHeader_1x02_P2.54mm_Vertical, symbol Connector_Generic:Conn_01x02
- added On/Off_Switch1: Conn_01x03, Connector_PinHeader_2.54mm:PinHeader_1x03_P2.54mm_Vertical, symbol Connector_Generic:Conn_01x03
Connections:
- net 3.3: no longer HR_Sensor1.4 (Pin_4), IMU_R1.5 (Pin_5), OLED1.2 (Pin_2), U1.JP6_4 (VCC_1), Vibration_Motor1.1 (Pin_1)
- net 3.7: now also HR_Sensor1.4 (Pin_4), IMU_R1.5 (Pin_5), OLED1.2 (Pin_2), U1.JP6_1 (RAW), Vibration_Motor1.1 (Pin_1), 3.7_Vias1.1 (Pin_1), 3.7_Vias1.2 (Pin_2), On/Off_Switch1.3 (Pin_3); no longer USBC1.1 (Pin_1), Voltage_Regulator1.1 (Pin_1)
- new net BAT: On/Off_Switch1.2 (Pin_2), USBC1.1 (Pin_1), Voltage_Regulator1.1 (Pin_1)
- no-connect marks 34 -> 35
